Commit message: urdf finish

File: urdf/manipulator.urdf (robot description, URDF)
Before this commit: robot ros_mani, 8 links, 7 joints
Links:
- added link mani_left_gear_support_link; visual mesh filename=package://ros_manipulator_project/meshes/MeshBody9.stl scale=0.002 0.002 0.002
- added link mani_left_gripper_link; visual mesh filename=package://ros_manipulator_project/meshes/MeshBody11.stl scale=0.002 0.002 0.002
- added link mani_right_gear_support_link; visual mesh filename=package://ros_manipulator_project/meshes/MeshBody10.stl scale=0.002 0.002 0.002
- added link mani_right_gripper_link; visual mesh filename=package://ros_manipulator_project/meshes/MeshBody12.stl scale=0.002 0.002 0.002
Joints:
- added joint gear_support_joint: type revolute, parent mani_gripper_base_link, child mani_left_gear_support_link, origin xyz=1.18 0.28 -0.21 rpy=1.57 0 0, axis 0 0 1, limit lower=0.0 upper=1.3 effort=1000.0 velocity=1.0, mimic joint=gripper_base_joint
- added joint gripper_joint: type revolute, parent mani_left_gear_link, child mani_left_gripper_link, origin xyz=0.15 -0.6 -0.1 rpy=0 0 0.42, axis 0 0 -1, limit lower=0.0 upper=1.3 effort=1000.0 velocity=1.0, mimic joint=gripper_base_joint
- added joint sub_gear_support_joint: type revolute, parent mani_gripper_base_link, child mani_right_gear_support_link, origin xyz=1.18 0.28 -0.005 rpy=0 0 0, axis 0 1 0, limit lower=0.0 upper=1.3 effort=1000.0 velocity=1.0, mimic joint=gear_support_joint
- added joint sub_gripper_joint: type revolute, parent mani_right_gear_link, child mani_right_gripper_link, origin xyz=0.23 0.1 0.57 rpy=1.57 0.32 0, axis 0 0 1, limit lower=0.0 upper=1.3 effort=1000.0 velocity=1.0, mimic joint=gripper_joint
- joint gripper_base_joint: limit lower=0.0 upper=3.1416 effort=1000.0 velocity=1.0 -> lower=0.0 upper=1.3 effort=1000.0 velocity=1.0; origin xyz=0.1 -0.3 -0.55 rpy=1.57 0 0 -> xyz=0.8 0.28 -0.4 rpy=1.57 0 0
- joint sub_gripper_base_joint: limit lower=0.0 upper=3.1416 effort=1000.0 velocity=1.0 -> lower=0.0 upper=1.3 effort=1000.0 velocity=1.0; origin xyz=0 0.5 0 rpy=0 0 0 -> xyz=0.77 0.28 0.15 rpy=0 0 0
