Commit message: urdf, teensy_code 수정

File: urdf/manipulator_v3.urdf (robot description, URDF)
Before this commit: robot ros_mani, 12 links, 11 joints
Joints:
- joint arm01_joint: axis 0 0 1 -> 1 0 0; origin xyz=0.0335 0.238 0 rpy=0 3.1416 1 -> xyz=0.0015 0.238 0 rpy=0 3.1416 0
- joint arm02_joint: origin xyz=-0.01 0.18 0.015 rpy=1.57 0 0 -> xyz=0.018 0.18 0.015 rpy=1.57 0 0
- joint arm03_joint: origin xyz=0.01 -0.03 -0.055 rpy=1.57 3.1416 0 -> xyz=0.01 -0.03 -0.055 rpy=1.57 1.57 0
- joint lid_joint: axis 0 0 1 -> 1 0 0; origin xyz=-0.007 0.025 0.083 rpy=0 1.57 0 -> xyz=-0.007 0.025 0.083 rpy=1.57 0 0
